File: HW/vfd.kicad_pcb (KiCad board)
At the start: 2 copper layers, 101.5 x 25.5 mm, 49 parts, among them Q1 2N7002, Q2 Si2319CDS, Q3 2N7002, Q4 Si2319CDS, Q5 2N7002, Q6 2N7002, T1 Transformer_1P_1S, U1 HCS-12SS59T, U2 MCP1663, U3 MCP1663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

Commit message: added esp and battery foo
Parts:
- added C14: 1u, Capacitor_SMD:C_0805_2012Metric, F.Cu at (213.3, 31.9)
- added C19: 1u, Capacitor_SMD:C_0805_2012Metric, F.Cu at (223.0, 25.1)
- added C20: 100n, Capacitor_SMD:C_0603_1608Metric, F.Cu at (222.8, 26.8)
- added C21: 1u, Capacitor_SMD:C_0805_2012Metric, F.Cu at (213.3, 33.8)
- added C22: 100n, Capacitor_SMD:C_0603_1608Metric, F.Cu at (213.1, 35.5)
- added D3: led, LED_SMD:LED_0603_1608Metric, F.Cu at (216.5, 31.7)
- added R14: 1k, Resistor_SMD:R_0603_1608Metric, F.Cu at (226.2, 24.9)
- added R17: 1k5, Resistor_SMD:R_0603_1608Metric, F.Cu at (213.1, 37.0)
- added R18: 10k, Resistor_SMD:R_0603_1608Metric, F.Cu at (216.5, 33.2)
- added U5: TP4056, Package_SO:SO-8_5.3x6.2mm_P1.27mm, F.Cu at (216.4, 27.5)
- added U6: ESP32-wroom-32, vfd:ESP-wroom-32, F.Cu at (233.7, 80.0)
