File: HW/vfd.sch (KiCad schematic (older format))
At the start: 8 parts, among them U1 HCS-12SS59T

Commit message: added heater schmeatic
Parts:
- added Q? (x2): BC547, Package_TO_SOT_THT:TO-92_Inline, symbol Transistor_BJT:BC547
- added Q? (x2): BC557, Package_TO_SOT_THT:TO-92_Inline, symbol Transistor_BJT:BC557
- added R? (x4): 220, symbol Device:R_Small
- added T?: Transformer_1P_1S, symbol Device:Transformer_1P_1S
Connections:
- net labels added: +3.3V, GPIO15, GPIO16
- wire segments 14 -> 30
Changed lines of the file:
@@
 Text GLabel 2650 1550 0    50   Input ~ 0
 F-
-Wire Wire Line
-	3400 1050 4300 1050
 $Comp
 L Device:R_Small R2
 U 1 1 5BA8FE52
-P 4300 950
-F 0 "R2" H 4359 996 50  0000 L CNN
-F 1 "8k2" H 4359 905 50  0000 L CNN
-F 2 "Resistors_SMD:R_0603" H 4300 950 50  0001 C CNN
-F 3 "~" H 4300 950 50  0001 C CNN
-	1    4300 950
+P 3800 900
+F 0 "R2" H 3859 946 50  0000 L CNN
+F 1 "8k2" H 3859 855 50  0000 L CNN
+F 2 "Resistors_SMD:R_0603" H 3800 900 50  0001 C CNN
+F 3 "~" H 3800 900 50  0001 C CNN
+	1    3800 900
 	1    0    0    -1
 $EndComp
@@
 L Device:C_Small C5
 U 1 1 5BA8FEC5
-P 4300 1150
-F 0 "C5" H 4392 1196 50  0000 L CNN
-F 1 "82p" H 4392 1105 50  0000 L CNN
-F 2 "Capacitors_SMD:C_0603" H 4300 1150 50  0001 C CNN
-F 3 "~" H 4300 1150 50  0001 C CNN
-	1    4300 1150
-	1    0    0    -1
-$EndComp
-Connection ~ 4300 1050
+P 3800 1200
+F 0 "C5" H 3892 1246 50  0000 L CNN
+F 1 "82p" H 3892 1155 50  0000 L CNN
+F 2 "Capacitors_SMD:C_0603" H 3800 1200 50  0001 C CNN
+F 3 "~" H 3800 1200 50  0001 C CNN
+	1    3800 1200
+	1    0    0    -1
+$EndComp
 $Comp
 L power:GND #PWR0102
 U 1 1 5BA8FF49
-P 4300 1250
-F 0 "#PWR0102" H 4300 1000 50  0001 C CNN
-F 1 "GND" H 4305 1077 50  0000 C CNN
-F 2 "" H 4300 1250 50  0001 C CNN
-F 3 "" H 4300 1250 50  0001 C CNN
-	1    4300 1250
+P 3800 1300
+F 0 "#PWR0102" H 3800 1050 50  0001 C CNN
+F 1 "GND" H 3805 1127 50  0000 C CNN
+F 2 "" H 3800 1300 50  0001 C CNN
+F 3 "" H 3800 1300 50  0001 C CNN
+	1    3800 1300
 	1    0    0    -1
 $EndComp
@@
 L power:+5V #PWR0103
 U 1 1 5BA9001E
-P 4300 850
-F 0 "#PWR0103" H 4300 700 50  0001 C CNN
-F 1 "+5V" H 4315 1023 50  0000 C CNN
-F 2 "" H 4300 850 50  0001 C CNN
-F 3 "" H 4300 850 50  0001 C CNN
-	1    4300 850
+P 3800 800
+F 0 "#PWR0103" H 3800 650 50  0001 C CNN
+F 1 "+5V" H 3815 973 50  0000 C CNN
+F 2 "" H 3800 800 50  0001 C CNN
+F 3 "" H 3800 800 50  0001 C CNN
+	1    3800 800
 	1    0    0    -1
 $EndComp
@@
 	1    0    0    -1
 $EndComp
+Wire Wire Line
+	3400 1050 3800 1050
+Wire Wire Line
+	3800 1000 3800 1050
+Wire Wire Line
+	3800 1100 3800 1050
+Connection ~ 3800 1050
+$Comp
+L Transistor_BJT:BC547 Q?
+U 1 1 5BA922CE
+P 5000 1700
+F 0 "Q?" H 5191 1746 50  0000 L CNN
+F 1 "BC547" H 5191 1655 50  0000 L CNN
+F 2 "Package_TO_SOT_THT:TO-92_Inline" H 5200 1625 50  0001 L CIN
+F 3 "http://www.fairchildsemi.com/ds/BC/BC547.pdf" H 5000 1700 50  0001 L CNN
+	1    5000 1700
+	1    0    0    -1
+$EndComp
+$Comp
+L Transistor_BJT:BC547 Q?
+U 1 1 5BA92395
+P 6150 1700
+F 0 "Q?" H 6340 1746 50  0000 L CNN
+F 1 "BC547" H 6340 1655 50  0000 L CNN
+F 2 "Package_TO_SOT_THT:TO-92_Inline" H 6350 1625 50  0001 L CIN
+F 3 "http://www.fairchildsemi.com/ds/BC/BC547.pdf" H 6150 1700 50  0001 L CNN
+	1    6150 1700
+	-1   0    0    -1
+$EndComp
+$Comp
+L Transistor_BJT:BC557 Q?
+U 1 1 5BA927D3
+P 6150 1200
+F 0 "Q?" H 6340 1154 50  0000 L CNN
+F 1 "BC557" H 6340 1245 50  0000 L CNN
+F 2 "Package_TO_SOT_THT:TO-92_Inline" H 6350 1125 50  0001 L CIN
+F 3 "http://www.fairchildsemi.com/ds/BC/BC557.pdf" H 6150 1200 50  0001 L CNN
+	1    6150 1200
+	-1   0    0    1
+$EndComp
+$Comp
+L Transistor_BJT:BC557 Q?
+U 1 1 5BA92884
+P 5000 1200
+F 0 "Q?" H 5191 1154 50  0000 L CNN
+F 1 "BC557" H 5191 1245 50  0000 L CNN
+F 2 "Package_TO_SOT_THT:TO-92_Inline" H 5200 1125 50  0001 L CIN
+F 3 "http://www.fairchildsemi.com/ds/BC/BC557.pdf" H 5000 1200 50  0001 L CNN
+	1    5000 1200
+	1    0    0    1
+$EndComp
+Wire Wire Line
+	6050 1000 6050 800
+Wire Wire Line
+	6050 800  5100 800
+Wire Wire Line
+	5100 1000 5100 800
+Connection ~ 5100 800
+Wire Wire Line
+	5100 800  4950 800
+Wire Wire Line
+	6050 2500 5100 2500
+Connection ~ 5100 2500
+Wire Wire Line
+	5100 2500 4950 2500
+Wire Wire Line
+	5100 1400 5100 1450
+Connection ~ 5100 1450
+Wire Wire Line
+	5100 1450 5100 1500
+$Comp
+L power:+3.3V #PWR?
+U 1 1 5BA94086
+P 4950 800
+F 0 "#PWR?" H 4950 650 50  0001 C CNN
+F 1 "+3.3V" H 4965 973 50  0000 C CNN
+F 2 "" H 4950 800 50  0001 C CNN
+F 3 "" H 4950 800 50  0001 C CNN
+	1    4950 800
+	1    0    0    -1
+$EndComp
+$Comp
+L power:GND #PWR?
+U 1 1 5BA94111
+P 4950 2500
+F 0 "#PWR?" H 4950 2250 50  0001 C CNN
+F 1 "GND" H 4955 2327 50  0000 C CNN
+F 2 "" H 4950 2500 50  0001 C CNN
+F 3 "" H 4950 2500 50  0001 C CNN
+	1    4950 2500
+	1    0    0    -1
+$EndComp
+Wire Wire Line
+	6050 1400 6050 1450
+Connection ~ 6050 1450
+Wire Wire Line
+	6050 1450 6050 1500
+$Comp
+L Device:Transformer_1P_1S T?
+U 1 1 5BA9483E
+P 5600 1850
+F 0 "T?" V 5554 2090 50  0000 L CNN
+F 1 "Transformer_1P_1S" V 5645 2090 50  0000 L CNN
+F 2 "" H 5600 1850 50  0001 C CNN
+F 3 "~" H 5600 1850 50  0001 C CNN
+	1    5600 1850
+	0    1    1    0
+$EndComp
+Wire Wire Line
+	5100 1450 5400 1450
+Wire Wire Line
+	5800 1450 6050 1450
+Text GLabel 5400 2250 3    50   Input ~ 0
+F-
+Text GLabel 5800 2250 3    50   Input ~ 0
+F+
+$Comp
+L Device:R_Small R?
+U 1 1 5BA95794
+P 4700 1200
+F 0 "R?" V 4504 1200 50  0000 C CNN
+F 1 "220" V 4595 1200 50  0000 C CNN
+F 2 "" H 4700 1200 50  0001 C CNN
+F 3 "~" H 4700 1200 50  0001 C CNN
+	1    4700 1200
+	0    1    1    0
+$EndComp
+$Comp
+L Device:R_Small R?
+U 1 1 5BA9581F
+P 6450 1700
+F 0 "R?" V 6254 1700 50  0000 C CNN
+F 1 "220" V 6345 1700 50  0000 C CNN
+F 2 "" H 6450 1700 50  0001 C CNN
+F 3 "~" H 6450 1700 50  0001 C CNN
+	1    6450 1700
+	0    1    1    0
+$EndComp
+$Comp
+L Device:R_Small R?
+U 1 1 5BA9588E
+P 4700 1700
+F 0 "R?" V 4504 1700 50  0000 C CNN
+F 1 "220" V 4595 1700 50  0000 C CNN
+F 2 "" H 4700 1700 50  0001 C CNN
+F 3 "~" H 4700 1700 50  0001 C CNN
+	1    4700 1700
+	0    1    1    0
+$EndComp
+$Comp
+L Device:R_Small R?
+U 1 1 5BA9592B
+P 6450 1200
+F 0 "R?" V 6254 1200 50  0000 C CNN
+F 1 "220" V 6345 1200 50  0000 C CNN
+F 2 "" H 6450 1200 50  0001 C CNN
+F 3 "~" H 6450 1200 50  0001 C CNN
+	1    6450 1200
+	0    1    1    0
+$EndComp
+Text GLabel 4600 1200 0    50   Input ~ 0
+GPIO15
+Text GLabel 6550 1700 2    50   Input ~ 0
+GPIO16
+Text GLabel 4600 1700 0    50   Input ~ 0
+GPIO15
+Text GLabel 6550 1200 2    50   Input ~ 0
+GPIO16
+Wire Wire Line
+	5100 1900 5100 2500
+Wire Wire Line
+	6050 1900 6050 2500
 $EndSCHEMATC

Commit message: added stepups, setdown, battery
Parts:
- removed C3: 10u, symbol Device:CP_Small
- removed C4: 4u7, symbol Device:CP_Small
- removed Q? (x2): BC547, Package_TO_SOT_THT:TO-92_Inline, symbol Transistor_BJT:BC547
- removed Q? (x2): BC557, Package_TO_SOT_THT:TO-92_Inline, symbol Transistor_BJT:BC557
- added BT1: Battery_Cell, Battery:BatteryHolder_Keystone_1042_1x18650, symbol Device:Battery_Cell
- added C10, C12, C17, C18, C3, C9, C? (x2): 1u, Capacitor_SMD:C_0805_2012Metric, symbol Device:C_Small
- added C11, C13, C15, C16, C4, C6, C8: 100n, Capacitor_SMD:C_0603_1608Metric, symbol Device:C_Small
- added C7: TBD, Capacitor_SMD:C_0603_1608Metric, symbol Device:C_Small
- added D1, D2: D_Schottky, Diode_SMD:D_SMA, symbol Device:D_Schottky
- added D?: led, symbol Device:LED_Small
- added L1, L2, L3: 15u, Inductor_SMD:L_Taiyo-Yuden_MD-4040, symbol Device:L
- added Q1, Q3, Q5, Q6: 2N7002, Package_TO_SOT_SMD:SOT-23, symbol Transistor_FET:2N7002
- added Q2, Q4: Si2319CDS, Package_TO_SOT_SMD:SOT-23, symbol Transistor_FET:Si2319CDS
- added R10, R7: 47, Resistor_SMD:R_0603_1608Metric, symbol Device:R_Small
- added R11: TBD, Resistor_SMD:R_0603_1608Metric, symbol Device:R_Small
- added R12: 25k, Resistor_SMD:R_0603_1608Metric, symbol Device:R_Small
- added R13, R16: 1k, Resistor_SMD:R_0603_1608Metric, symbol Device:R_Small
- added R15: 3k, Resistor_SMD:R_0603_1608Metric, symbol Device:R_Small
- added R8, R9: 10k, Resistor_SMD:R_0603_1608Metric, symbol Device:R_Small
- added R?: 1k, symbol Device:R_Small
- added R?: 1k5, symbol Device:R_Small
- added SW?: SW_DIP_x01, symbol Switch:SW_DIP_x01
- added U2, U3: MCP1663, Package_TO_SOT_SMD:SOT-23-5, symbol vfd:MCP1663
- added U4: LM3670MF, Package_TO_SOT_SMD:SOT-23-5, symbol Regulator_Switching:LM3670MF
- added U?: TP4056, symbol vfd:TP4056
- C1: footprint Capacitors_SMD:C_0805 -> Capacitor_SMD:C_0805_2012Metric
- C2, C5: footprint Capacitors_SMD:C_0603 -> Capacitor_SMD:C_0603_1608Metric
- R1, R2: footprint Resistors_SMD:R_0603 -> Resistor_SMD:R_0603_1608Metric
- R3, R4, R5, R6: renamed from R?; value 220 -> 47; footprint (none) -> Resistor_SMD:R_0603_1608Metric
- T1: renamed from T?; footprint (none) -> vfd:SRF0703
Connections:
- net labels added: VBAT, VBAT_SW, VUSB
- wire segments 30 -> 97
Other:
- note added: "Todo:\nESP\nAkku + schaltung\nUSB-seriell\nOtter\n"
- note removed: "Todo:\nFilamentspannung\nESP\n36V\nAkku + schaltung\nUSB-seriell\nOtter\n"

Commit message: added esp and battery foo
Parts:
- added C20, C22: 100n, Capacitor_SMD:C_0603_1608Metric, symbol Device:C_Small
- added C21: 1u, Capacitor_SMD:C_0805_2012Metric, symbol Device:C_Small
- added R18: 10k, Resistor_SMD:R_0603_1608Metric, symbol Device:R_Small
- added U6: ESP32-wroom-32, vfd:ESP-wroom-32, symbol vfd:ESP32-wroom-32
- D3: renamed from D?; footprint (none) -> LED_SMD:LED_0603_1608Metric
- R14, R17: renamed from R?; footprint (none) -> Resistor_SMD:R_0603_1608Metric
- U5: renamed from U?; footprint (none) -> Package_SO:SO-8_5.3x6.2mm_P1.27mm
- gave numbers to parts that had none: 3
Connections:
- net labels added: EN
- wire segments 97 -> 100
Other:
- note added: "Todo:\nESP\nUnterspannungsschutz\nUSB-seriell\nOtter\n"
- note removed: "Todo:\nESP\nAkku + schaltung\nUSB-seriell\nOtter\n"
